File: rp2040-board.kicad_pcb (KiCad board)
At the start: 4 copper layers, 105.3 x 75.1 mm, 157 parts, among them J1 24V IN, J10 E0-RUNOUT, J11 FAN1, J12 FAN2, J13 FAN3, J14 HB, J15 E0, J16 TH-E0, J17 X-STEPPER, J18 Y-STEPPER, J19 ZA-STEPPER, J2 USB4105-GF-A, J20 E0-STEPPER, J21 ZB-STEPPER, J3 PGA2040, J4 3_GPIO, J5 PROBE, J6 X-ENDSTOP, J7 TH-HB, J8 Y-ENDSTOP, J9 Z-ENDSTOP, Q1 AO3400C, Q2 AO3400C, Q3 AO3400C, U1 AMS1117-3.3, U2 TPS5450DDAR, U3 74HCT365D,653, U4 FDS8896, U5 FDS8896, U6 TMC2226-SA-T, U7 TMC2226-SA-T, U8 TMC2226-SA-T, U9 TMC2226-SA-T

Commit message: finished, for now, finally
Parts:
- added J22: Exp. Header 2, Connector_PinHeader_2.54mm:PinHeader_1x02_P2.54mm_Vertical, F.Cu at (198.9, 105.4)
- added J23: Exp. Header 3, Connector_PinHeader_2.54mm:PinHeader_1x02_P2.54mm_Vertical, F.Cu at (198.9, 108.3)
- J4: value 3_GPIO -> Exp. Header 1; footprint Connector_PinSocket_2.54mm:PinSocket_1x03_P2.54mm_Vertical -> Connector_PinHeader_2.54mm:PinHeader_1x02_P2.54mm_Vertical
- moved J4 9.44 mm to (198.9, 102.5), turned to -90 degrees
- moved R35 0.40 mm to (155.2, 94.7)
Connections:
- net Net-(J3-PadF8) renamed GPIO21
- net Net-(J3-PadG8) renamed GPIO20
- J3 pad B1: XDIR -> XEN
- J3 pad C2: XEN -> XDIR
- J3 pad D2: YDIR -> YEN
- J3 pad E2: YEN -> YDIR
- J3 pad F2: ZDIR -> ZEN
- J3 pad F7: Net-(J3-PadF7) -> GPIO22
- J3 pad G3: E0DIR -> E0EN
- J3 pad G4: E0EN -> E0DIR
- J3 pad H2: ZEN -> ZDIR
- R41 pad 2: XEN -> XENR
- R42 pad 2: YEN -> YENR
- R51 pad 2: E0EN -> E0ENR
- R52 pad 2: ZEN -> ZENR
- RN1 pad 1: XDIR -> XDIRR
- RN1 pad 2: XSTP -> XSTPR
- RN1 pad 3: XEN -> XENR
- RN2 pad 1: YDIR -> YDIRR
- RN2 pad 2: YSTP -> YSTPR
- RN2 pad 3: YEN -> YENR
- RN3 pad 1: ZDIR -> ZDIRR
- RN3 pad 2: ZSTP -> ZSTPR
- RN3 pad 3: ZEN -> ZENR
- RN4 pad 1: E0DIR -> E0DIRR
- RN4 pad 2: E0STP -> E0STPR
- RN4 pad 3: E0EN -> E0ENR
- U6 pad 20: XSTP -> XSTPR
- U6 pad 23: XDIR -> XDIRR
- U6 pad 5: XEN -> XENR
- U7 pad 20: YSTP -> YSTPR
- U7 pad 23: YDIR -> YDIRR
- U7 pad 5: YEN -> YENR
- U8 pad 20: E0STP -> E0STPR
- U8 pad 23: E0DIR -> E0DIRR
- U8 pad 5: E0EN -> E0ENR
- U9 pad 20: ZSTP -> ZSTPR
- U9 pad 23: ZDIR -> ZDIRR
- U9 pad 5: ZEN -> ZENR
Routing:
- net Net-(R35-Pad1): track 60.1 -> 199.7 mm, vias 8 -> 15
- net XSTOP: track 0.00 -> 99.5 mm, vias 0 -> 2
- net YSTOP: track 0.00 -> 76.5 mm, vias 0 -> 3
- net +5V: track 55.7 -> 127.0 mm, vias 3 -> 5
- net VCC: track 225.9 -> 155.3 mm, vias 9 -> 28
- net XSTP: track 17.9 -> 75.0 mm, vias 2 -> 1
- net +3.3V: track 298.9 -> 355.8 mm, vias 16 -> 19
- net GND: track 302.2 -> 245.7 mm, vias 56 -> 47
- net E0STOP: track 0.00 -> 55.8 mm, vias 0 -> 2
- net XEN: track 21.2 -> 74.6 mm
- net ZSTOP: track 0.00 -> 48.9 mm, vias 0 -> 4
- net XDIR: track 21.6 -> 69.9 mm, vias 2 -> 1
- net Net-(J2-PadA7): track 2.77 -> 44.4 mm, vias 0 -> 3
- net Net-(J2-PadA6): track 2.77 -> 44.3 mm, vias 0 -> 3
- net /E0_THERM: track 2.61 -> 43.4 mm, vias 0 -> 1
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- added copper zone on In2.Cu, net VCC
Other:
- board text added: "(PK is a bad influence) Party in the back!"
- board text added: "FriedSalmon2040 - Rev 1"
- board text added: "JLCJLCJLCJLC"
